File: src/PCB_LEDS/PCB_LEDS.kicad_sch (KiCad schematic)
At the start: 35 parts, among them J1 Conn_01x05, Q1 BC337, Q2 BC337, Q3 BC337

Commit message: Add files via upload
Other:
- note removed: "15x150mm"
- company: (none) -> ITS VILLADA
- title: (none) -> "A" Pillar LED ARRAY PCB
Changed lines of the file:
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@@
 (kicad_sch (version 20211123) (generator eeschema)
   (paper "A4")
+  (title_block
+    (title "\"A\" Pillar LED ARRAY PCB")
+    (date "2022-11-20")
+    (rev "3")
+    (company "ITS VILLADA")
+    (comment 1 "Designed By: Gaston Grasso")
+    (comment 2 "2022")
+  )
   (wire (pts (xy 213.36 92.71) (xy 213.36 83.82))
     (stroke (width 0) (type default) (color 0 0 0 0))
@@
     (stroke (width 0) (type default) (color 0 0 0 0))
   )
-  (text "15x150mm\n" (at 144.78 35.56 0)
-    (effects (font (size 1.27 1.27)) (justify left bottom))
-  )
   (global_label "LED_R" (shape input) (at 181.61 111.76 180) (fields_autoplaced)
